Commit message: separate control board

File: edy_dualarm_description/urdf/edy_dualarm_description.urdf (robot description, URDF)
Before this commit: robot edy_dualarm_description, 21 links, 20 joints
Links:
- link l_link_9: mass 0.00675806648920072 -> 0.0423839787748426
Joints:
- joint l_joint_8: origin xyz=0 0 0.04087 rpy=0 0 3.1416 -> xyz=0 0 0.039 rpy=0 0 3.1416
- joint l_joint_eef: origin xyz=0 0 0.07887 rpy=0 0 0 -> xyz=0 0 0.06739 rpy=0 0 0
