Commit message: add gazebo-related package for edy but model is still unstable and needed to be stablized by adjusting parameters i.e. PID

File: edy_dualarm_description/urdf/edy_dualarm_gazebo.urdf (robot description, URDF)
Before this commit: robot edy_dualarm_description, 21 links, 20 joints
Links:
- link root: geometry collision box size=0.001 0.001 0.001; visual box size=0.001 0.001 0.001
